Commit message: Added visuals and collisions

File: description/robot_core.xacro (robot description, xacro)
@@ -1,3 +1,97 @@
 <?xml version="1.0"?>
 <robot xmlns:xacro="http://www.ros.org/wiki/xacro" >
+    <material name="white">
+        <color rgba="1 1 1 1 "/>
+    </material>
+    <material name="orange">
+        <color rgba="1 0.3 0.1 1"/>
+    </material>
+    <material name="blue">
+        <color rgba="0.2 0.2 1 1"/>
+    </material>
+    <material name="black">
+        <color rgba="0 0 0 1"/>
+    </material>
+    <link name="base_link">
+    </link>
+    <!--Chassis Link-->
+    <joint name ="chassis_joint" type="fixed">
+        <parent link="base_link"/>
+        <child link="chassis"/>
+        <origin xyz ="-0.3 0 0"/>
+    </joint>
+    <link name = "chassis">
+        <visual>
+            <origin xyz="0.2 0 0.125"/>
+            <geometry>
+                <box size="0.4 0.4 .25"/>
+            </geometry>
+            <material name="white"/>
+        </visual>
+         <collision>
+            <origin xyz="0.2 0 0.125"/>
+            <geometry>
+                <box size="0.4 0.4 .25"/>
+            </geometry>
+        </collision>
+    </link>
+    <!-- Left Wheel Link-->
+    <joint name="left_wheel_joint" type="continuous">
+        <parent link="base_link"/>
+        <child link="left_wheel"/>
+        <origin xyz ="0 0.175 0" rpy="-${pi/2} 0 0"/>
+        <axis xyz="0 0 -1.5"/>
+    </joint>
+    <link name="left_wheel">
+        <visual>
+            <geometry>
+                <cylinder radius="0.05" length="0.03" />
+            </geometry>
+            <material name="blue"/>
+        </visual>
+          <collision>
+            <geometry>
+                <cylinder radius="0.05" length="0.03" />
+            </geometry>
+        </collision>
+    </link>
+    <!--Right Wheel Link-->
+    <joint name="right_wheel_joint" type="continuous">
+        <parent link="base_link"/>
+        <child link="right_wheel"/>
+        <origin xyz ="0 -0.175 0" rpy="${pi/2} 0 0"/>
+        <axis xyz="0 0 -1.5"/>
+    </joint>
+      <link name="right_wheel">
+        <visual>
+            <geometry>
+                <cylinder radius="0.05" length="0.03" />
+            </geometry>
+            <material name="blue"/>
+        </collision>
+              <visual>
+            <geometry>
+                <cylinder radius="0.05" length="0.03" />
+            </geometry>
+        </collision>
+    </link>
+    <!--Caster Wheel Link-->
+    <joint name="caster_wheel_joint" type="fixed">
+        <parent link="chassis"/>
+        <child link="caster_wheel_link"/>
+        <origin xyz ="0.28 0 0"/>
+    </joint>
+    <link name="caster_wheel">
+        <visual>
+            <geometry>
+                <sphere radius="0.05"/>
+            </geometry>
+            <material name="orange"/>
+        </visual>
+        <collision>
+            <geometry>
+                <sphere radius="0.05"/>
+            </geometry>
+        </collision>
+    </link>
 </robot>

Commit message: Fixed errors of caster_wheel_joint

File: description/robot_core.xacro (robot description, xacro)
@@ -29,5 +29,5 @@
             <material name="white"/>
         </visual>
-         <collision>
+        <collision>
             <origin xyz="0.2 0 0.125"/>
             <geometry>
@@ -50,5 +50,5 @@
             <material name="blue"/>
         </visual>
-          <collision>
+        <collision>
             <geometry>
                 <cylinder radius="0.05" length="0.03" />
@@ -63,12 +63,12 @@
         <axis xyz="0 0 -1.5"/>
     </joint>
-      <link name="right_wheel">
+    <link name="right_wheel">
         <visual>
             <geometry>
-                <cylinder radius="0.05" length="0.03" />
+                <cylinder radius="0.05" length="0.03"/>
             </geometry>
             <material name="blue"/>
-        </collision>
-              <visual>
+        </visual>
+        <collision>
             <geometry>
                 <cylinder radius="0.05" length="0.03" />
@@ -79,5 +79,5 @@
     <joint name="caster_wheel_joint" type="fixed">
         <parent link="chassis"/>
-        <child link="caster_wheel_link"/>
+        <child link="caster_wheel"/>
         <origin xyz ="0.28 0 0"/>
     </joint>

Commit message: Added the informations about the inertia

File: description/robot_core.xacro (robot description, xacro)
@@ -36,4 +36,7 @@
             </geometry>
         </collision>
+        <xacro:inertial_box mass="1.0" x="0.4" y="0.4" z="0.25">
+            <origin xyz="0.2 0 0.125" rpy="0 0 0"/>
+        </xacro:inertial_box>
     </link>
     <!-- Left Wheel Link-->
@@ -56,4 +59,7 @@
             </geometry>
         </collision>
+        <xacro:inertial_cylinder mass="0.5" length="0.03" radius="0.05">
+            <origin xyz="0 0 0" rpy="0 0 0"/>
+        </xacro:inertial_cylinder>
     </link>
     <!--Right Wheel Link-->
@@ -76,4 +82,7 @@
             </geometry>
         </collision>
+        <xacro:inertial_cylinder mass="0.5" length="0.03" radius="0.05">
+            <origin xyz="0 0 0" rpy="0 0 0"/>
+        </xacro:inertial_cylinder>
     </link>
     <!--Caster Wheel Link-->
@@ -95,4 +104,7 @@
             </geometry>
         </collision>
+        <xacro:inertial_sphere mass="0.2" radius="0.05">
+            <origin xyz="0 0 0" rpy="0 0 0"/>
+        </xacro:inertial_sphere>
     </link>
 </robot>

Commit message: Added the values of gazebo reference frame, fixed the caster wheels placement and added the value of two frictional force

File: description/robot_core.xacro (robot description, xacro)
@@ -1,7 +1,8 @@
 <?xml version="1.0"?>
-<robot xmlns:xacro="http://www.ros.org/wiki/xacro" >
+<robot xmlns:xacro="http://www.ros.org/wiki/xacro">
     <xacro:include filename="inertial_macros.xacro"/>
+    <!-- RViz colors -->
     <material name="white">
-        <color rgba="1 1 1 1 "/>
+        <color rgba="1 1 1 1"/>
     </material>
     <material name="orange">
@@ -14,17 +15,17 @@
         <color rgba="0 0 0 1"/>
     </material>
-    <link name="base_link">
-    </link>
-    <!--Chassis Link-->
-    <joint name ="chassis_joint" type="fixed">
+    <!-- Base link -->
+    <link name="base_link"></link>
+    <!-- Chassis -->
+    <joint name="chassis_joint" type="fixed">
         <parent link="base_link"/>
         <child link="chassis"/>
-        <origin xyz ="-0.3 0 0"/>
+        <origin xyz="-0.3 0 0"/>
     </joint>
-    <link name = "chassis">
+    <link name="chassis">
         <visual>
             <origin xyz="0.2 0 0.125"/>
             <geometry>
-                <box size="0.4 0.4 .25"/>
+                <box size="0.4 0.4 0.25"/>
             </geometry>
             <material name="white"/>
@@ -33,5 +34,5 @@
             <origin xyz="0.2 0 0.125"/>
             <geometry>
-                <box size="0.4 0.4 .25"/>
+                <box size="0.4 0.4 0.25"/>
             </geometry>
         </collision>
@@ -40,9 +41,16 @@
         </xacro:inertial_box>
     </link>
-    <!-- Left Wheel Link-->
+    <gazebo reference="chassis">
+        <material>
+            <ambient>1 1 1 1</ambient>
+            <diffuse>1 1 1 1</diffuse>
+            <specular>0.5 0.5 0.5 1</specular>
+        </material>
+    </gazebo>
+    <!-- Left wheel -->
     <joint name="left_wheel_joint" type="continuous">
         <parent link="base_link"/>
         <child link="left_wheel"/>
-        <origin xyz ="0 0.175 0" rpy="-${pi/2} 0 0"/>
+        <origin xyz="0 0.175 0" rpy="-${pi/2} 0 0"/>
         <axis xyz="0 0 -1.5"/>
     </joint>
@@ -50,5 +58,5 @@
         <visual>
             <geometry>
-                <cylinder radius="0.05" length="0.03" />
+                <cylinder radius="0.05" length="0.03"/>
             </geometry>
             <material name="blue"/>
@@ -56,5 +64,5 @@
         <collision>
             <geometry>
-                <cylinder radius="0.05" length="0.03" />
+                <cylinder radius="0.05" length="0.03"/>
             </geometry>
         </collision>
@@ -63,9 +71,16 @@
         </xacro:inertial_cylinder>
     </link>
-    <!--Right Wheel Link-->
+    <gazebo reference="left_wheel">
+        <material>
+            <ambient>0.2 0.2 1 1</ambient>
+            <diffuse>0.2 0.2 1 1</diffuse>
+            <specular>0.5 0.5 0.5 1</specular>
+        </material>
+    </gazebo>
+    <!-- Right wheel -->
     <joint name="right_wheel_joint" type="continuous">
         <parent link="base_link"/>
         <child link="right_wheel"/>
-        <origin xyz ="0 -0.175 0" rpy="${pi/2} 0 0"/>
+        <origin xyz="0 -0.175 0" rpy="${pi/2} 0 0"/>
         <axis xyz="0 0 -1.5"/>
     </joint>
@@ -79,5 +94,5 @@
         <collision>
             <geometry>
-                <cylinder radius="0.05" length="0.03" />
+                <cylinder radius="0.05" length="0.03"/>
             </geometry>
         </collision>
@@ -86,9 +101,16 @@
         </xacro:inertial_cylinder>
     </link>
-    <!--Caster Wheel Link-->
+    <gazebo reference="right_wheel">
+        <material>
+            <ambient>0.2 0.2 1 1</ambient>
+            <diffuse>0.2 0.2 1 1</diffuse>
+            <specular>0.5 0.5 0.5 1</specular>
+        </material>
+    </gazebo>
+    <!-- Caster wheel -->
     <joint name="caster_wheel_joint" type="fixed">
         <parent link="chassis"/>
         <child link="caster_wheel"/>
-        <origin xyz ="0.28 0 0"/>
+        <origin xyz="0.15 0 0"/>
     </joint>
     <link name="caster_wheel">
@@ -108,3 +130,12 @@
         </xacro:inertial_sphere>
     </link>
+    <gazebo reference="caster_wheel">
+        <material>
+            <ambient>1 0.3 0.1 1</ambient>
+            <diffuse>1 0.3 0.1 1</diffuse>
+            <specular>0.5 0.5 0.5 1</specular>
+        </material>
+        <mu1 value="0.001"/>
+        <mu2 value="0.001"/>
+    </gazebo>
 </robot>
