Commit message: Edited the config

File: description/lidar.xacro (robot description, xacro)
@@ -4,5 +4,5 @@
     <parent link="chassis"/>
     <child link="laser_link"/>
-    <origin xyz="0.1 0 0.175" rpy="0 0 0"/>
+    <origin xyz="0.4 0 0.27" rpy="0 0 0"/>
   </joint>
   <link name="laser_link">
@@ -31,13 +31,14 @@
         <scan>
           <horizontal>
-            <samples>720</samples>
+            <samples>360</samples>
             <resolution>1</resolution>
-            <min_angle>-1.5708</min_angle>
-            <max_angle>1.5708</max_angle>
+            <min_angle>-3.14</min_angle>
+            <max_angle>3.14</max_angle>
           </horizontal>
         </scan>
         <range>
-          <min>0.1</min>
-          <max>10.0</max>
+          <min>0.3</min>
+          <max>12.0</max>
+          <resolution>0.01</resolution>
         </range>
       </ray>

Commit message: updated

File: description/lidar.xacro (robot description, xacro)
@@ -18,5 +18,4 @@
       </geometry>
     </collision>
-    <!-- Only one inertial_cylinder call is needed -->
     <xacro:inertial_cylinder mass="0.2" length="0.1" radius="0.05">
         <origin xyz="0 0 0" rpy="0 0 0"/>
@@ -26,5 +25,5 @@
     <sensor name="laser" type="ray">
       <pose>0 0 0 0 0 0</pose>
-      <visualize>true</visualize>
+      <visualize>false</visualize>
       <update_rate>10</update_rate>
       <ray>
@@ -45,8 +44,7 @@
       <plugin name="laser_controller" filename="libgazebo_ros_ray_sensor.so">
         <ros>
-            <argument>/out:=scan</argument>
+            <remapping>scan:=scan</remapping>
         </ros>
-        <output_type>sensor_msgs/LaserScan</output_type>
-        <frame name="laser_link"/>
+        <frame_name>laser_link</frame_name>
       </plugin>
     </sensor>

File: description/robot.urdf.xacro (robot description, xacro)
@@ -3,4 +3,5 @@
  <xacro:include filename="robot_core.xacro" />
  <xacro:include filename="gazebo_control.xacro" />
- <xacro:include filename="lidar.xacro"/>
+ <xacro:include filename="lidar.xacro" />
+ <xacro:include filename="camera.xacro"/>
 </robot>

File: description/robot_core.xacro (robot description, xacro)
@@ -53,5 +53,5 @@
         <child link="left_wheel"/>
         <origin xyz="0 0.175 0" rpy="-${pi/2} 0 0"/>
-        <axis xyz="0 0 -1.5"/>
+        <axis xyz="0 0 -1"/>
     </joint>
     <link name="left_wheel">
@@ -83,5 +83,5 @@
         <child link="right_wheel"/>
         <origin xyz="0 -0.175 0" rpy="${pi/2} 0 0"/>
-        <axis xyz="0 0 -1.5"/>
+        <axis xyz="0 0 -1"/>
     </joint>
     <link name="right_wheel">
